File: pcb/LKP-Chu-Electrode-Tile/LKP-Chu-Electrode-Tile.kicad_pcb (KiCad board)
At the start: 2 copper layers, 216 x 90 mm, 20 parts, among them J1 Intercon, J10 Electrode 0, J11 Electrode 2, J12 Electrode 4, J13 Electrode 6, J14 Electrode 8, J15 Electrode 10, J16 Electrode 12, J17 Electrode 14, J2 Electrode 1, J3 Electrode 3, J4 Electrode 5, J5 Electrode 7, J6 Electrode 9, J7 Electrode 11, J8 Electrode 13, J9 Electrode 15

Commit message: Add dimension PDFs for easier reference
Other:
- board text added: "Edge to Connector Center"

Commit message: Also update LKP-Chu-Electrode-Tile.
Other:
- net class CapSense removed
- net class Default removed

Commit message: Bump versions for LKP-Chu-Electrode-Tile.
Other:
- board text added: "LKP-Chu Electrode Tile 2x8 V1.1"
- board text removed: "LKP-Chu Electrode Tile 2x8 V1.0"
Changed lines of the file:
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@@
   )
   (paper "A4")
+  (title_block
+    (title "LKP Chu Electrode Tile")
+    (rev "1.1")
+  )
   (layers
     (0 "F.Cu" signal)
@@
   (gr_line (start 40.25 41) (end 40.25 131) (layer "Edge.Cuts") (width 0.1))
   (gr_line (start 40.25 131) (end 256.25 131) (layer "Edge.Cuts") (width 0.1))
-  (gr_text "LKP-Chu Electrode Tile\n2x8 V1.0" (at 152.25 86) (layer "B.SilkS")
+  (gr_text "LKP-Chu Electrode Tile\n2x8 V1.1" (at 152.25 86) (layer "B.SilkS")
     (effects (font (size 1.5 1.5) (thickness 0.3)) (justify mirror))
   )

Commit message: v4.2
Unify export settings across projects
Other:
- rule pad_to_mask_clearance: 0.051 -> 0
Changed lines of the file:
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@@
   )
   (setup
-    (pad_to_mask_clearance 0.051)
-    (solder_mask_min_width 0.25)
+    (stackup
+      (layer "F.SilkS" (type "Top Silk Screen"))
+      (layer "F.Paste" (type "Top Solder Paste"))
+      (layer "F.Mask" (type "Top Solder Mask") (thickness 0.01))
+      (layer "F.Cu" (type "copper") (thickness 0.035))
+      (layer "dielectric 1" (type "core") (thickness 1.51) (material "FR4") (epsilon_r 4.5) (loss_tangent 0.02))
+      (layer "B.Cu" (type "copper") (thickness 0.035))
+      (layer "B.Mask" (type "Bottom Solder Mask") (thickness 0.01))
+      (layer "B.Paste" (type "Bottom Solder Paste"))
+      (layer "B.SilkS" (type "Bottom Silk Screen"))
+      (copper_finish "None")
+      (dielectric_constraints no)
+    )
+    (pad_to_mask_clearance 0)
     (grid_origin 61.25 63.5)
     (pcbplotparams
-      (layerselection 0x00010fc_ffffffff)
+      (layerselection 0x00010f0_ffffffff)
       (plot_on_all_layers_selection 0x0000000_00000000)
       (disableapertmacros false)
-      (usegerberextensions false)
-      (usegerberattributes false)
-      (usegerberadvancedattributes false)
+      (usegerberextensions true)
+      (usegerberattributes true)
+      (usegerberadvancedattributes true)
       (creategerberjobfile false)
       (dashed_line_dash_ratio 12.000000)
@@
       (outputformat 1)
       (mirror false)
-      (drillshape 1)
+      (drillshape 0)
       (scaleselection 1)
-      (outputdirectory "")
+      (outputdirectory "out/")
     )
   )
