File: pcb/LKP-Diva-Electrode-Tile/LKP-Diva-Electrode-Tile.kicad_pcb (KiCad board)
At the start: 2 copper layers, 258 x 40 mm, 19 parts, among them J1 Intercon, J10 Electrode 0, J11 Electrode 2, J12 Electrode 4, J13 Electrode 6, J14 Electrode 8, J15 Electrode 10, J16 Electrode 12, J17 Electrode 14, J2 Electrode 1, J3 Electrode 3, J4 Electrode 5, J5 Electrode 7, J6 Electrode 9, J7 Electrode 11, J8 Electrode 13, J9 Electrode 15

Commit message: Add dimension PDFs for easier reference
Other:
- board text added: "Edge to Connector Center"

Commit message: LKP-Diva-Electrode-Tile: Update to new format.
- Update hatched fill.
- Increase the electrode size to 14.6x39mm.
- Change routing to fit the new pad size.
- Bump version number.
Parts:
- J10, J11, J12, J13, J14, J15, J16, J17, J2, J3, J4, J5, J6, J7, J8, J9: footprint private:CapSense_Electrode_14x38mm -> private:CapSense_Electrode_14.6x39mm
Routing:
- net Net-(J1-Pad16): track 8.51 -> 7.47 mm
- net Net-(J1-Pad15): track 14.5 -> 13.9 mm
- net Net-(J1-Pad11): track 77.0 -> 76.4 mm
- net Net-(J1-Pad7): track 139.5 -> 138.9 mm
- net Net-(J1-Pad3): track 201.9 -> 201.4 mm
- net Net-(J1-Pad9): track 108.2 -> 107.7 mm
- net Net-(J1-Pad5): track 170.7 -> 170.2 mm
- net Net-(J1-Pad10): track 98.4 -> 97.9 mm
- net Net-(J1-Pad6): track 160.9 -> 160.4 mm
- net GNDA: vias 30 -> 0
- removed copper zone on F.Cu, net GNDA
Other:
- net class CapSense removed
- net class Default removed
- board text added: "LKP-Diva Electrode Tile 1x16 V1.1"
- board text removed: "LKP-Diva Electrode Tile 1x16 V1.0"

Commit message: v4.2
Unify export settings across projects
Other:
- rule pad_to_mask_clearance: 0.051 -> 0
Changed lines of the file:
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@@
   )
   (setup
-    (pad_to_mask_clearance 0.051)
-    (solder_mask_min_width 0.25)
+    (stackup
+      (layer "F.SilkS" (type "Top Silk Screen"))
+      (layer "F.Paste" (type "Top Solder Paste"))
+      (layer "F.Mask" (type "Top Solder Mask") (thickness 0.01))
+      (layer "F.Cu" (type "copper") (thickness 0.035))
+      (layer "dielectric 1" (type "core") (thickness 1.51) (material "FR4") (epsilon_r 4.5) (loss_tangent 0.02))
+      (layer "B.Cu" (type "copper") (thickness 0.035))
+      (layer "B.Mask" (type "Bottom Solder Mask") (thickness 0.01))
+      (layer "B.Paste" (type "Bottom Solder Paste"))
+      (layer "B.SilkS" (type "Bottom Silk Screen"))
+      (copper_finish "None")
+      (dielectric_constraints no)
+    )
+    (pad_to_mask_clearance 0)
     (grid_origin 281.25 124)
     (pcbplotparams
