File: pcb/LKP-IF-QC/LKP-IF-QC.kicad_pcb (KiCad board)
At the start: 2 copper layers, 41 x 36 mm, 9 parts, among them J1 JST SH, J2 JST SH, J3 LKP SWD .1" Extra Long, J4 LKP I/O .1" Extra Long, J5 INT Passthrough, U1 TCA9406DCTR

Commit message: v4.2
Unify export settings across projects
Changed lines of the file:
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@@
       (plot_on_all_layers_selection 0x0000000_00000000)
       (disableapertmacros false)
-      (usegerberextensions false)
+      (usegerberextensions true)
       (usegerberattributes true)
       (usegerberadvancedattributes true)
-      (creategerberjobfile true)
+      (creategerberjobfile false)
       (dashed_line_dash_ratio 12.000000)
       (dashed_line_gap_ratio 3.000000)
@@
     (pad "4" smd roundrect (at 1.5 -2 270) (size 0.6 1.55) (layers "F.Cu" "F.Paste" "F.Mask") (roundrect_rratio 0.25)
       (net 4 "/SCL_A") (pinfunction "Pin_4") (pintype "passive"))
-    (pad "MP" smd roundrect (at -2.8 1.875 270) (size 1.2 1.8) (layers "F.Cu" "F.Paste" "F.Mask") (roundrect_rratio 0.208333))
-    (pad "MP" smd roundrect (at 2.8 1.875 270) (size 1.2 1.8) (layers "F.Cu" "F.Paste" "F.Mask") (roundrect_rratio 0.208333))
+    (pad "MP" smd roundrect (at -2.8 1.875 270) (size 1.2 1.8) (layers "F.Cu" "F.Paste" "F.Mask") (roundrect_rratio 0.2083333333))
+    (pad "MP" smd roundrect (at 2.8 1.875 270) (size 1.2 1.8) (layers "F.Cu" "F.Paste" "F.Mask") (roundrect_rratio 0.2083333333))
     (model "${KICAD6_3DMODEL_DIR}/Connector_JST.3dshapes/JST_SH_SM04B-SRSS-TB_1x04-1MP_P1.00mm_Horizontal.wrl"
       (offset (xyz 0 0 0))
@@
     (pad "4" smd roundrect (at 1.5 -2 90) (size 0.6 1.55) (layers "F.Cu" "F.Paste" "F.Mask") (roundrect_rratio 0.25)
       (net 4 "/SCL_A") (pinfunction "Pin_4") (pintype "passive"))
-    (pad "MP" smd roundrect (at -2.8 1.875 90) (size 1.2 1.8) (layers "F.Cu" "F.Paste" "F.Mask") (roundrect_rratio 0.208333))
-    (pad "MP" smd roundrect (at 2.8 1.875 90) (size 1.2 1.8) (layers "F.Cu" "F.Paste" "F.Mask") (roundrect_rratio 0.208333))
+    (pad "MP" smd roundrect (at -2.8 1.875 90) (size 1.2 1.8) (layers "F.Cu" "F.Paste" "F.Mask") (roundrect_rratio 0.2083333333))
+    (pad "MP" smd roundrect (at 2.8 1.875 90) (size 1.2 1.8) (layers "F.Cu" "F.Paste" "F.Mask") (roundrect_rratio 0.2083333333))
     (model "${KICAD6_3DMODEL_DIR}/Connector_JST.3dshapes/JST_SH_SM04B-SRSS-TB_1x04-1MP_P1.00mm_Horizontal.wrl"
       (offset (xyz 0 0 0))
